File: O2 Macrodevice Nucleo Board KiCad/Nucleo_L476RG/Nucleo_L476RG.kicad_sch (KiCad schematic)
At the start: 12 parts, among them J1 TS-108-T-A-1, J2 TS-108-T-A-1, U1 STM32L476RGTx, X1 ABS25-32.768KHZ-6-T

Commit message: updated NFC and Nucleo boards with new SMD header connectors
Parts:
- removed J1, J2: TS-108-T-A-1, CON8_1X8_TUC_HTS_SAI, symbol Header_Connector:TS-108-T-A-1
- added J3, J4, J5: 61000418221, 61000418221_WRE, symbol SMD Header:61000418221
Connections:
- net GND: now also J3.4, J5.3
- net GPIO_EXTIO: now also J5.2
- net MISO: now also J4.4
- net MOSI: now also J4.3
- net SCK: now also J5.1
- net SPI1_NSS: now also J3.2
- net SWCLK: now also J3.3
- net SWDIO: now also J4.1
- net TX_TP: now also J4.2
- net at C1.2, C2.2, C27.2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: now also J3.1
